Commit message: Viidennen luennon korjaukset

File: src/r3_2020/urdf/r3_2020.urdf (robot description, URDF)
Before this commit: robot r3_2020, 5 links, 4 joints
Links:
- added link sonar1_link, mass 0.030; collision box size=0.01 0.1 0.01; visual box size=0.01 0.05 0.01
Joints:
- removed joint wheel_left_link
- added joint sonar1_joint: type fixed, parent base_link, child sonar1_link, origin xyz=-0.235 0 0.16 rpy=0 0 3.14, axis 0 0 0
- added joint wheel_left_joint: type continuous, parent base_link, child wheel_left_link, origin xyz=0 0 0 rpy=0 0 0, axis 0 -1 0
